File: bill_acceptor/interface/ict_to_hid.sch (EAGLE design)
At the start: 12 parts, among them J14 TC2030-CC2538-BL, J15 MICRO_USB_B_HIROSE_ZX62R-B-5P, U1 ATUM, U2 FT232RQ

Commit message: routed version
Parts:
- removed C4: 10u, SparkFun:CAP_POL1206
- removed J14: TC2030-CC2538-BL, connector:TC2030-CC2538-BL
- removed L1: (no value), SparkFun:INDUCTOR0603
- removed R4: 2k, rcl:R-US_R0603
- removed R5: 1.5k, rcl:R-US_R0603
- added H1, H2, H3, H4: MOUNT-HOLE3.2, holes:MOUNT-HOLE3.2
- added J2: SCREW-TERMINAL_2_0.100, headers:SCREW-TERMINAL_2_0.100
- added J3: (no value), pinhead:PINHD-1X5
- added J4: TC2030-CC2538-BL, connector:TC2030-CC2538-BL
- added R2: 1.5k, passives:RESISTOR0603_RES
- added R3: 2k, passives:RESISTOR0603_RES
- C1: value 0.1u -> 10nF; device rcl:C-EUC0603 -> passives:CAPACITOR0603_CAP; DIGIKEY 445-1316-1-ND -> (none)
- C2, C3: value 0.1u -> 4.7uF; device rcl:C-EUC0603 -> passives:CAPACITOR0603_CAP; DIGIKEY 445-1316-1-ND -> (none)
- R1: device rcl:R-US_R0603 -> passives:RESISTOR0603_RES
- U2: value FT232RQ -> MAX8887EZK33+T; device ftdichip:FT232RQ -> chips:MAX8887EZK33+T; DIGIKEY 768-1008-1-ND -> (none)
- renumbered J15 to J1
Connections:
- removed net N$6: C2.1, C4.+, L1.2, U2.VCC
- new net N$5: C1.1, U2.BP
- net !RESET: now also J4.!RESET, U1.!RESET; no longer J14.!RESET
- net BOOTLOADER_CTRL: now also J4.BL_CTRL, U1.BTLDR_CTRL; no longer J14.BL_CTRL
- net BOOTLOADER_RX: now also J4.RX, U1.BTLDR_RX; no longer J14.RX
- net BOOTLOADER_TX: now also J4.TX, U1.BTLDR_TX; no longer J14.TX
- net GND: now also J3.5, J4.GND, R3.1; no longer C4.-, J14.GND, R4.1, U2.GND@1, U2.GND@2, U2.TEST
- net ICT_PULSE+: now also J2.1, J3.3
- net ICT_PULSE-: now also J2.2, J3.4, R3.2; no longer R4.2
- net N$12: now also R2.1; no longer R5.1
- net USB5V: now also C2.1, J3.2, U2.!SHDN, U2.IN; no longer C1.1, L1.1
- net VCC: now also J3.1, J4.VCC, R2.2, U2.OUT; no longer J14.VCC, R5.2, U2.3V3OUT, U2.VCCIO
Other:
- note removed: "3V3 Regulator"
- moved on the sheet: R1
